File: circuit-ai-frontend/public/demo/usb_esp32_sensor.kicad_pcb (KiCad board)
At the start: 2 copper layers, 60 x 40 mm, 8 parts, among them J1 USB-C, U1 ESP32, U2 LDO_3V3, U3 BME280

Commit message: Auto-save: Daily system backup 2026-04-19 00:00:09
Parts:
- J1: footprint Connector_USB:USB_C_Receptacle_USB2.0 -> Connector_USB:USB_C_Receptacle
- moved U1 4.00 mm to (34.0, 20.0)
- moved C2 2.24 mm to (23.0, 28.0)
- moved C1 2.00 mm to (20.0, 28.0)
- moved R1 2.00 mm to (45.0, 28.0)
- moved R2 2.00 mm to (48.0, 28.0)
Routing:
- net GND: track 44.0 -> 0.00 mm, vias 0 -> 1
- net SCL: track 0.00 -> 27.7 mm
- net SDA: track 0.00 -> 25.8 mm
- net +3V3: track 32.0 -> 54.4 mm, vias 0 -> 1
- net ALERT: track 0.00 -> 17.7 mm
- net VIN: track 4.00 -> 11.5 mm
- added copper zone on B.Cu, net GND
- added copper zone on F.Cu, net GND
Other:
- outline, holes or cut-outs redrawn
- board text added: "CIRCUIT.AI"
- board text added: "REV A"
- board text added: "USB ESP32 SENSOR"
