File: hardware/reference_designs/spi_flash_adapter_v1/spi_flash_adapter_v1.kicad_pcb (KiCad board)
At the start: 2 copper layers, 90 x 50 mm, 33 parts, among them J1 HOST_SPI_1x06, U1 TXU0304PWR, U2 W25Q128JWSIQ, U3 TLV75518PDBVR

Commit message: Harden SPI adapter startup and ground reference
Parts:
- added JP1: ENABLE_AFTER_RAIL_CHECK, Connector_PinHeader_2.54mm:PinHeader_1x02_P2.54mm_Vertical, F.Cu at (147.0, 98.0)
- added R5: 10k, Resistor_SMD:R_0603_1608Metric, F.Cu at (133.0, 94.0)
- added R6: 10k, Resistor_SMD:R_0603_1608Metric, F.Cu at (161.0, 85.0)
- added R7: 10k, Resistor_SMD:R_0603_1608Metric, F.Cu at (151.0, 100.0)
- added TP16: TRANSLATOR_OE, TestPoint:TestPoint_Pad_D1.5mm, F.Cu at (155.0, 101.0)
- added TP17: GND, TestPoint:TestPoint_Pad_D1.5mm, F.Cu at (146.0, 93.0)
- added TP18: GND, TestPoint:TestPoint_Pad_D1.5mm, F.Cu at (175.0, 101.0)
- H1, H2, H3, H4: footprint MountingHole_3.2mm_M3 -> MountingHole:MountingHole_3.2mm_M3
Connections:
- U1 pad 8: /DUT_1V8 -> /TRANSLATOR_OE
Routing:
- net /GND: track 147.1 -> 17.3 mm, vias 7 -> 20
- net /DUT_1V8: track 85.7 -> 137.2 mm, vias 5 -> 0
- net /HOST_3V3: track 23.3 -> 68.6 mm
- net /TRANSLATOR_OE: track 0.00 -> 20.6 mm
- net /DUT_CS_N: track 33.1 -> 26.5 mm, vias 2 -> 0
- net /DUT_IO3_HOLD_N: track 19.7 -> 15.2 mm
- net /DUT_MOSI: track 35.4 -> 31.2 mm
- net /HOST_MOSI: track 43.3 -> 39.2 mm
- net /DUT_SCLK: track 35.3 -> 33.4 mm, vias 3 -> 0
- net /HOST_CS_N: track 44.6 -> 42.9 mm, vias 2 -> 0
- net /HOST_MISO: track 47.0 -> 45.7 mm, vias 2 -> 0
- net /DUT_MISO: track 29.1 -> 29.8 mm, vias 3 -> 0
- net /HOST_SCLK: track 39.4 -> 38.8 mm
- net /3V3: track 55.7 -> 56.3 mm
- net /DUT_IO2_WP_N: track 18.7 -> 19.1 mm, vias 3 -> 0
- added copper zone on B.Cu, net /GND
- added copper zone on F.Cu, net /GND
Other:
- board text added: "ENABLE AFTER RAIL CHECK + CS HIGH"
- board text added: "HS SPI FLASH ADAPTER v1 REV 0.2"
- board text added: "JP1 OPEN AT POWER UP/DOWN"
- board text removed: "HS SPI FLASH ADAPTER v1"
